File: RESISTORS.kicad_sch (KiCad schematic)
At the start: 10 parts

Commit message: Fix minor problem.
Signed-off-by: John Bradley <flypie@rocketmail.com>
Changed lines of the file:
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@@
       (effects (font (size 1.27 1.27)) hide)
     )
-    (property "Value" "" (id 1) (at 46.99 91.4399 90)
+    (property "Value" "GND" (id 1) (at 46.99 91.4399 90)
       (effects (font (size 1.27 1.27)) (justify right))
     )
